Commit message: changed cube to rectangular wall

File: data/rectangle_horizontal_half.urdf (robot description, URDF)
Before this commit: robot rectangle, 1 links, 0 joints
Links:
- link base_link: geometry collision box size=0.4 0.1 1; visual box size=0.4 0.1 1

File: data/rectangle_vertical_half.urdf (robot description, URDF)
Before this commit: robot rectangle, 1 links, 0 joints
Links:
- link base_link: geometry collision box size=0.4 0.1 1; visual box size=0.4 0.1 1
